File: KiCad/Line Following Robot.kicad_pcb (KiCad board)
At the start: 2 copper layers, 130.5 x 169.5 mm, 20 parts, among them SW1 SW_Push, U1 5V Buck Convertor, U2 ESP32-S3-DEVKITC-1-N8R8, U3 6V Buck Convertor, U4 IR Sensor Array, U5 Motor Driver, U7 Battery

Commit message: fixed pcb
Routing:
- net GND: track 665.7 -> 625.2 mm
- net /VCC: track 281.8 -> 267.8 mm
- net /M4: track 85.5 -> 84.0 mm

Commit message: fixed pcb
Routing:
- net /5V: track 339.1 -> 254.0 mm, vias 0 -> 3
- net /6V: track 233.3 -> 209.4 mm, vias 0 -> 1
- net /IR4: track 150.1 -> 143.5 mm
- net /VCC: track 267.8 -> 264.4 mm

Commit message: added step file
Parts:
- removed ?: , 
- removed C3: 100 nF, Line Following Robot:Capacitor
- removed REF** (x4): MountingHole_2.2mm_M2, MountingHole:MountingHole_2.2mm_M2
- removed REF** (x3): MountingHole_4mm, MountingHole:MountingHole_4mm
Connections:
- A1 pad 5: +3V3 -> /3V3
- A2 pad 5: +3V3 -> /3V3
- U2 pad J1_1: Net-(U2-3V3) -> /3V3
- U2 pad J1_2: unconnected-(U2-3V3.-PadJ1_2) -> /3V3IR
- U4 pad 11: /5V -> /3V3IR
- U5 pad 11: unconnected-(U5-EEP-Pad11) -> /3V3
Routing:
- net /3V3: track 0.00 -> 165.8 mm, vias 0 -> 1
- net /3V3IR: track 0.00 -> 122.7 mm, vias 0 -> 1
- net /5V: track 254.0 -> 160.5 mm, vias 3 -> 6
- net +3V3: track 75.8 -> 0.00 mm
- net Net-(U2-3V3): track 59.0 -> 0.00 mm, vias 2 -> 0
- net /IR_MAIN: track 156.1 -> 157.3 mm
