File: KiCad/Line Following Robot.kicad_pcb (KiCad board)
At the start: 2 copper layers, 130.5 x 169.5 mm, 18 parts, among them SW1 SW_Push, U1 5V Buck Convertor, U2 ESP32-S3-DEVKITC-1-N8R8, U3 6V Buck Convertor, U4 IR Sensor Array, U5 Motor Driver, U7 Battery

Commit message: fixed everything
Parts:
- removed the REF** at (60.9, 154.1)
- removed the REF** at (102.1, 61.4)
- removed the REF** at (143.5, 171.4)
- removed the REF** at (102.0, 37.3)
- removed the REF** at (60.9, 171.4)
- removed the REF** at (143.5, 154.1)
- removed the REF** at (102.0, 23.8)
- removed SW1: SW_Push, Button_Switch_THT:SW_PUSH_6mm
- removed U5: Motor Driver, Line Following Robot:Motor Driver
- added REF**: MountingHole_2.2mm_M2, MountingHole:MountingHole_2.2mm_M2, F.Cu at (102.5, 63.5)
- added REF**: MountingHole_2.2mm_M2, MountingHole:MountingHole_2.2mm_M2, F.Cu at (102.5, 23.0)
- added REF**: MountingHole_2.2mm_M2, MountingHole:MountingHole_2.2mm_M2, F.Cu at (142.4, 154.1)
- added REF**: MountingHole_2.2mm_M2, MountingHole:MountingHole_2.2mm_M2, F.Cu at (142.4, 171.4)
- added REF**: MountingHole_2.2mm_M2, MountingHole:MountingHole_2.2mm_M2, F.Cu at (61.7, 154.1)
- added REF**: MountingHole_2.2mm_M2, MountingHole:MountingHole_2.2mm_M2, F.Cu at (61.7, 171.4)
- added REF**: MountingHole_2.2mm_M2, MountingHole:MountingHole_2.2mm_M2, F.Cu at (102.5, 44.7)
- added SW2: SW_SPDT, Button_Switch_THT:SW_Slide-03_Wuerth-WS-SLTV_10x2.5x6.4_P2.54mm, F.Cu at (161.6, 142.4)
- added U6: ~, aeronexus:PinHeader_1x08_P2.54mm_Vertical, F.Cu at (82.5, 96.8)
Routing:
- net /VCC: track 263.2 -> 152.2 mm, vias 0 -> 2
- net /3V3IR: track 122.7 -> 205.1 mm
- net /M3: track 79.5 -> 121.1 mm, vias 0 -> 2
- net /MDIN1: track 16.1 -> 56.5 mm
- net /MDIN2: track 21.9 -> 62.3 mm
- net GND: track 617.7 -> 653.8 mm
- net Net-(U6-GND-Pad11): track 0.00 -> 35.8 mm, vias 0 -> 2
- net /M2: track 70.5 -> 98.4 mm, vias 0 -> 4
- net /IN4: track 48.2 -> 26.1 mm
- net /M1: track 68.9 -> 90.9 mm, vias 0 -> 2
- net /M4: track 84.0 -> 102.2 mm, vias 0 -> 2
- net /IN3: track 49.8 -> 32.1 mm
- net /3V3: track 165.8 -> 183.3 mm, vias 1 -> 2
- net /6V: track 209.0 -> 191.9 mm
- net Net-(SW2-A): track 58.6 -> 67.5 mm
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- added copper zone on B.Cu, net GND
- added copper zone on F.Cu, net GND

Commit message: fixed pcb and schematic
Parts:
- removed the REF** at (102.5, 63.5)
- removed the REF** at (142.4, 154.1)
- removed the REF** at (61.7, 171.4)
- added REF**: MountingHole_2.2mm_M2, MountingHole:MountingHole_2.2mm_M2, F.Cu at (61.7, 171.4)
- added REF**: MountingHole_2.2mm_M2, MountingHole:MountingHole_2.2mm_M2, F.Cu at (102.5, 63.5)
- added REF**: MountingHole_2.2mm_M2, MountingHole:MountingHole_2.2mm_M2, F.Cu at (142.4, 154.0)
Connections:
- U6 pad 11: Net-(U6-GND-Pad11) -> GND
- U6 pad 16: Net-(U6-GND-Pad11) -> GND
- U6 pad 8: Net-(U6-GND-Pad11) -> GND
Routing:
- net GND: track 653.8 -> 698.0 mm, vias 1 -> 11
- net Net-(U6-GND-Pad11): track 35.8 -> 0.00 mm, vias 2 -> 0
- net /6V: track 191.9 -> 195.9 mm
- net /IR3: track 138.6 -> 140.7 mm
- net /IR2: track 152.7 -> 154.6 mm
- net /IR4: track 147.4 -> 148.3 mm
- net /3V3: track 183.3 -> 184.1 mm
- net /3V3IR: track 205.1 -> 204.3 mm
- net /MDIN2: track 62.3 -> 62.9 mm
- net /MDIN1: track 56.5 -> 57.0 mm
