File: KiCad/Line Following Robot.kicad_sch (KiCad schematic)
At the start: 12 parts, among them SW1 SW_Push, U1 5V Buck Convertor, U2 ESP32-S3-DEVKITC-1-N8R8, U3 6V Buck Convertor, U4 IR Sensor Array, U5 Motor Driver, U7 Battery

Commit message: added step file
Parts:
- removed C3: 100 nF, Line Following Robot:Capacitor, symbol Device:C
Connections:
- net +3V3 is gone; now on net 3V3: A1.5 (Encoder+), A2.5 (Encoder+)
- net 5V: no longer U4.11 (VCC)
- net 3V3: now reaches U2.J1_1 (3V3)
- net 3V3: now also U5.11 (EEP)
- net 3V3IR: now reaches U2.J1_2 (3V3.)
- net 3V3IR: now also U4.11 (VCC)
- no-connect marks 30 -> 28

Commit message: fixed everything
Parts:
- removed SW1: SW_Push, Button_Switch_THT:SW_PUSH_6mm, symbol Switch:SW_Push
- removed U5: Motor Driver, Line Following Robot:Motor Driver, symbol Line Following Robot:DRV8833_Dual_Motor_Driver_1.5A
- added SW2: SW_SPDT, Button_Switch_THT:SW_Slide-03_Wuerth-WS-SLTV_10x2.5x6.4_P2.54mm, symbol Switch:SW_SPDT
- added U6: ~, aeronexus:PinHeader_1x08_P2.54mm_Vertical, symbol Line Following Robot:DRV8833_Dual_Motor_Driver_1.5A
Connections:
- net 3V3: now also U6.4 (STBY)
- net 6V: now also U6.9 (VM)
- net IN3: now also U6.5 (BIN1)
- net IN4: now also U6.6 (BIN2)
- net M1: now also U6.12 (AO1)
- net M2: now also U6.13 (AO2)
- net M3: now also U6.14 (BO2)
- net M4: now also U6.15 (BO1)
- net MDIN1: now also U6.3 (AIN1)
- net MDIN2: now also U6.2 (AIN2)
- net VCC: now also SW2.2 (B)
- net at U7.1 (+): now also SW2.1 (A)
- new net: U6.11 (GND), U6.16 (GND), U6.8 (GND)
- no-connect marks 28 -> 31

Commit message: fixed pcb and schematic
Connections:
- net GND: now also U6.11 (GND), U6.16 (GND), U6.8 (GND)
Changed lines of the file:
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@@
+	)
+	(junction
+		(at 137.16 73.66)
+		(diameter 0)
+		(color 0 0 0 0)
 	)
 	(junction
@@
 	(wire
 		(pts
+			(xy 137.16 73.66) (xy 125.73 73.66)
+		)
+		(stroke
+			(width 0)
+			(type default)
+		)
+	)
+	(wire
+		(pts
 			(xy 233.68 137.16) (xy 243.84 137.16)
 		)
@@
 	(wire
 		(pts
-			(xy 146.05 73.66) (xy 125.73 73.66)
+			(xy 146.05 73.66) (xy 137.16 73.66)
 		)
 		(stroke
@@
 					(unit 1)
 				)
+			)
+		)
+	)
+	(symbol
+		(lib_id "power:GND")
+		(at 137.16 73.66 0)
+		(unit 1)
+		(exclude_from_sim no)
+		(in_bom yes)
+		(on_board yes)
+		(dnp no)
+		(fields_autoplaced yes)
+		(property "Reference" "#PWR09"
+			(at 137.16 80.01 0)
+			(effects
+				(font
+					(size 1.27 1.27)
+				)
+				(hide yes)
+			)
+		)
+		(property "Value" "GND"
+			(at 137.16 78.74 0)
+			(effects
+				(font
+					(size 1.27 1.27)
+				)
+			)
+		)
+		(property "Footprint" ""
+			(at 137.16 73.66 0)
+			(effects
+				(font
+					(size 1.27 1.27)
+				)
+				(hide yes)
+			)
+		)
+		(property "Datasheet" ""
+			(at 137.16 73.66 0)
+			(effects
+				(font
+					(size 1.27 1.27)
+				)
+				(hide yes)
+			)
+		)
+		(property "Description" "Power symbol creates a global label with name \"GND\" , ground"
+			(at 137.16 73.66 0)
+			(effects
+				(font
+					(size 1.27 1.27)
+				)
+				(hide yes)
+			)
+		)
+		(pin "1"
+		)
+		(instances
+			(project ""
+				(path "/251d369d-29e6-4cc4-9ad2-9627e3bfe5fc"
+					(reference "#PWR09")
+					(unit 1)
+				)
